Commit message: feat(validation): Pinocchio 3.9 cross-check via nanobind binding
Phase 4 acceptance: FK and Jacobian (LOCAL / WORLD / LOCAL_WORLD_ALIGNED)
agree with Pinocchio 3.9.0 to ~1e-15 (machine precision) on every fixture
URDF, over 1000 random configurations from a fixed seed. CLAUDE.md \xc2\xa711 demands
1e-10; we are at e-15.

Pieces:
- src/bindings/main.cpp: minimal nanobind module (_tinyspatial). Exposes
  Model accessors, build_model_from_urdf_file, forward_kinematics (returns
  list of 4x4 matrices), compute_jacobian (returns 6 x nv ndarray).
- python/tinyspatial/__init__.py: re-exports the extension.
- tests/validation/test_kinematics.py: loads each URDF in both libraries,
  samples 1000 random configurations via pin.randomConfiguration (fixed
  seed), compares FK at every joint and Jacobians at the last movable joint
  in all three reference frames. Applies a 6 x 6 row permutation to convert
  Pinocchio's linear-first Jacobian rows to our angular-first convention
  (documented in PINOCCHIO_PARITY.md, not a bug).
- tests/validation/requirements.txt: pip-install spec. Pins
  cmeel-urdfdom < 5 alongside pin==3.9.0 to avoid the urdfdom 6.x ABI break
  that masquerades as a missing liburdfdom_sensor.so.4.0.
- CMakeLists.txt: TINYSPATIAL_BUILD_VALIDATION=ON pulls in nanobind, builds
  the _tinyspatial extension into python/tinyspatial/, and registers a
  CTest entry under label 'pinocchio_parity' so
  'ctest --preset=validation -L pinocchio_parity' passes.
- tinyspatial_urdf static lib gets POSITION_INDEPENDENT_CODE for linkage
  into the shared extension.
- Fixture URDFs grew <limit> elements on every <joint type="revolute">,
  required by urdfdom (and harmless for us).
- docs/PINOCCHIO_PARITY.md generated: first parity table.

Standalone debug build remains untouched (92/92 tests still green, no
new compiler warnings, clang-format / clang-tidy clean).

Co-Authored-By: Claude Opus 4.7 <noreply@anthropic.com>

File: data/robots/franka_fr3.urdf (robot description, URDF)
Before this commit: robot franka_fr3, 8 links, 7 joints
Joints:
- joint fr3_joint1: limit (none) -> lower=-3.14159 upper=3.14159 effort=100 velocity=2.0
- joint fr3_joint2: limit (none) -> lower=-3.14159 upper=3.14159 effort=100 velocity=2.0
- joint fr3_joint3: limit (none) -> lower=-3.14159 upper=3.14159 effort=100 velocity=2.0
- joint fr3_joint4: limit (none) -> lower=-3.14159 upper=3.14159 effort=100 velocity=2.0
- joint fr3_joint5: limit (none) -> lower=-3.14159 upper=3.14159 effort=100 velocity=2.0
- joint fr3_joint6: limit (none) -> lower=-3.14159 upper=3.14159 effort=100 velocity=2.0
- joint fr3_joint7: limit (none) -> lower=-3.14159 upper=3.14159 effort=100 velocity=2.0

File: data/robots/simple_arm.urdf (robot description, URDF)
Before this commit: robot simple_arm, 3 links, 2 joints
Joints:
- joint joint1: limit (none) -> lower=-3.14159 upper=3.14159 effort=100 velocity=2.0
- joint joint2: limit (none) -> lower=-3.14159 upper=3.14159 effort=100 velocity=2.0

File: data/robots/so_arm101.urdf (robot description, URDF)
Before this commit: robot so_arm101, 7 links, 6 joints
Joints:
- joint elbow: limit (none) -> lower=-3.14159 upper=3.14159 effort=100 velocity=2.0
- joint shoulder_lift: limit (none) -> lower=-3.14159 upper=3.14159 effort=100 velocity=2.0
- joint shoulder_pan: limit (none) -> lower=-3.14159 upper=3.14159 effort=100 velocity=2.0
- joint wrist_pitch_joint: limit (none) -> lower=-3.14159 upper=3.14159 effort=100 velocity=2.0
- joint wrist_roll_joint: limit (none) -> lower=-3.14159 upper=3.14159 effort=100 velocity=2.0

File: data/robots/ur5e.urdf (robot description, URDF)
Before this commit: robot ur5e, 7 links, 6 joints
Joints:
- joint elbow_joint: limit (none) -> lower=-3.14159 upper=3.14159 effort=100 velocity=2.0
- joint shoulder_lift_joint: limit (none) -> lower=-3.14159 upper=3.14159 effort=100 velocity=2.0
- joint shoulder_pan_joint: limit (none) -> lower=-3.14159 upper=3.14159 effort=100 velocity=2.0
- joint wrist_1_joint: limit (none) -> lower=-3.14159 upper=3.14159 effort=100 velocity=2.0
- joint wrist_2_joint: limit (none) -> lower=-3.14159 upper=3.14159 effort=100 velocity=2.0
- joint wrist_3_joint: limit (none) -> lower=-3.14159 upper=3.14159 effort=100 velocity=2.0
